File: step/step-left/step-left-bottom.kicad_pcb (KiCad board)
At the start: 2 copper layers, 136.6 x 92.2 mm, 9 parts

Commit message: chore: Rename
Parts:
- G***: footprint Keebio-Art:Keebio-TwoTone -> natsukium-Art:natsukium-TwoTone
- REF**: footprint Keebio-Parts:VIA-0.6mm -> natsukium-Parts:VIA-0.6mm
Changed lines of the file:
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@@
       (drillshape 0)
       (scaleselection 1)
-      (outputdirectory ../gerbers/fourier-left-bottom/))
+      (outputdirectory ../gerbers/step-left-bottom/))
   )
   (net 0 "")
@@
     (pad 1 np_thru_hole circle (at 0 0) (size 2.2 2.2) (drill 2.2) (layers *.Cu *.Mask))
   )
-  (module Keebio-Parts:VIA-0.6mm (layer F.Cu)
+  (module natsukium-Parts:VIA-0.6mm (layer F.Cu)
     (at 74.6 66.225)
     (fp_text reference REF** (at 0 1.4) (layer F.SilkS) hide
@@
       (net 1 GND) (zone_connect 2))
   )
-  (module Keebio-Art:Keebio-TwoTone (layer B.Cu)
+  (module natsukium-Art:natsukium-TwoTone (layer B.Cu)
     (at 78.58125 61.317188 180)
     (fp_text reference G*** (at 0 0 180) (layer B.SilkS) hide
