File: step/step-right/step-right-bottom.kicad_pcb (KiCad board)
At the start: 2 copper layers, 141.4 x 92.2 mm, 8 parts

Commit message: chore: Rename
Parts:
- G***: footprint Keebio-Art:Keebio-TwoTone -> natsukium-Art:natsukium-TwoTone
Changed lines of the file:
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@@
       (drillshape 0)
       (scaleselection 1)
-      (outputdirectory ../gerbers/fourier-right-bottom))
+      (outputdirectory ../gerbers/step-right-bottom))
   )
   (net 0 "")
@@
     (pad 1 np_thru_hole circle (at 0 0) (size 2.2 2.2) (drill 2.2) (layers *.Cu *.Mask))
   )
-  (module Keebio-Art:Keebio-TwoTone (layer B.Cu)
+  (module natsukium-Art:natsukium-TwoTone (layer B.Cu)
     (at 90.7 78.575 180)
     (fp_text reference G*** (at 0 0 180) (layer B.SilkS) hide
