File: step/step-right/step-right.kicad_pcb (KiCad board)
At the start: 2 copper layers, 129.2 x 80.4 mm, 145 parts, among them J1 VCC, J3 RGB, J6 C6, J7 GND, U1 ProMicro, U2 TRRS

Commit message: chore: Rename
Parts:
- D_A1, D_A2, D_A3, D_A4, D_A5, D_A6, D_A7, D_B1, D_B2, D_B3, D_B4, D_B5, D_B7, D_C1, D_C3, D_C4, D_C5, D_C6, D_C7, D_D1, D_D2, D_D4, D_D5, D_D6, D_D7: footprint Keebio-Parts:Diode-Hybrid-Back -> natsukium-Parts:Diode-Hybrid-Back
- G***: footprint Keebio-Art:Keebio-TwoTone -> natsukium-Art:natsukium-TwoTone
- G***: footprint Keebio-Art:AIRI-Logo2 -> natsukium-Art:AIRI-Logo2
- G***: footprint Keebio-Art:Fourier-Rect -> natsukium-Art:Step-Rect
- G***: footprint Keebio-Art:Fourier-1.2 -> natsukium-Art:Step-1.2
- J1, J3, J6, J7, W2: footprint Keebio-Parts:Single-Pad -> natsukium-Parts:Single-Pad
- REF** (x65): footprint Keebio-Parts:VIA-0.6mm -> natsukium-Parts:VIA-0.6mm
- SW_RST1: footprint Keebio-Parts:SW_Tactile_SPST_Angled_MJTP1117 -> natsukium-Parts:SW_Tactile_SPST_Angled_MJTP1117
- U1: footprint Keebio-Parts:ArduinoProMicro-ZigZag -> natsukium-Parts:ArduinoProMicro-ZigZag
- U2: footprint Keebio-Parts:TRRS-PJ-320A -> natsukium-Parts:TRRS-PJ-320A
