File: step/step-right/step-right.sch (KiCad schematic (older format))
At the start: 72 parts, among them J1 VCC, J3 RGB, J6 C6, J7 GND, U1 ProMicro, U2 TRRS

Commit message: chore: Rename
Parts:
- D_A1, D_A2, D_A3, D_A4, D_A5, D_A6, D_A7, D_B1, D_B2, D_B3, D_B4, D_B5, D_B7, D_C1, D_C3, D_C4, D_C5, D_C6, D_C7, D_D1, D_D2, D_D4, D_D5, D_D6, D_D7: footprint Keebio-Parts:Diode-Hybrid-Back -> natsukium-Parts:Diode-Hybrid-Back
- J1, J3, J6, J7, W2: footprint Keebio-Parts:Single-Pad -> natsukium-Parts:Single-Pad; symbol fourier-right-rescue:TEST_1P-RESCUE-fourier-right -> step-right-rescue:TEST_1P-RESCUE-step-right
- SW_A1, SW_A2, SW_A3, SW_A4, SW_A5, SW_A6, SW_A7, SW_Ab7, SW_B1, SW_B2, SW_B3, SW_B4, SW_B5, SW_B7, SW_Bb7, SW_C1, SW_C3, SW_C4, SW_C5, SW_C6, SW_C7, SW_Cb6, SW_Cb7, SW_Cc7, SW_D1, SW_D2, SW_D4, SW_D5, SW_D6, SW_D7, SW_Db1, SW_Db4, SW_Db5, SW_Db6, SW_Db7, SW_Dc1, SW_Dc5, SW_Dc6, SW_Dc7: symbol fourier-right-rescue:SW_PUSH-RESCUE-fourier-right -> step-right-rescue:SW_PUSH-RESCUE-step-right
- SW_RST1: footprint Keebio-Parts:SW_Tactile_SPST_Angled_MJTP1117 -> natsukium-Parts:SW_Tactile_SPST_Angled_MJTP1117; symbol fourier-right-rescue:SW_PUSH-RESCUE-fourier-right -> step-right-rescue:SW_PUSH-RESCUE-step-right
- U1: footprint Keebio-Parts:ArduinoProMicro-ZigZag -> natsukium-Parts:ArduinoProMicro-ZigZag; symbol fourier-right-rescue:ProMicro-promicro -> step-right-rescue:ProMicro-promicro
- U2: footprint Keebio-Parts:TRRS-PJ-320A -> natsukium-Parts:TRRS-PJ-320A
